File: gpu-sync/11bitcount.sch (KiCad schematic (older format))
At the start: 3 parts, among them U1 74AC161, U2 74AC161, U3 74AC161

Commit message: gpu sync board component placement
Parts:
- U1, U2, U3: footprint (none) -> Package_DIP:DIP-16_W7.62mm_Socket_LongPads
Changed lines of the file:
@@
 $Descr A4 11693 8268
 encoding utf-8
-Sheet 2 7
+Sheet 4 7
 Title ""
 Date ""
@@
 AR Path="/5CC1878B/5CC1EE8E" Ref="U2"  Part="1"
 AR Path="/5CC8DF11/5CC1EE8E" Ref="U5"  Part="1"
-F 0 "U2" V 6300 3150 50  0000 C CNN
+F 0 "U5" V 6300 3150 50  0000 C CNN
 F 1 "74AC161" V 6100 3650 50  0000 C CNN
-F 2 "" H 6100 3650 50  0001 C CNN
+F 2 "Package_DIP:DIP-16_W7.62mm_Socket_LongPads" H 6100 3650 50  0001 C CNN
 F 3 "http://www.ti.com/lit/gpn/sn74LS161" H 6100 3650 50  0001 C CNN
 	1    6100 3650
@@
 AR Path="/5CC1878B/5CC1EE94" Ref="U1"  Part="1"
 AR Path="/5CC8DF11/5CC1EE94" Ref="U4"  Part="1"
-F 0 "U1" V 8100 3150 50  0000 C CNN
+F 0 "U4" V 8100 3150 50  0000 C CNN
 F 1 "74AC161" V 7900 3650 50  0000 C CNN
-F 2 "" H 7900 3650 50  0001 C CNN
+F 2 "Package_DIP:DIP-16_W7.62mm_Socket_LongPads" H 7900 3650 50  0001 C CNN
 F 3 "http://www.ti.com/lit/gpn/sn74LS161" H 7900 3650 50  0001 C CNN
 	1    7900 3650
@@
 AR Path="/5CC1878B/5CC1EEEE" Ref="U3"  Part="1"
 AR Path="/5CC8DF11/5CC1EEEE" Ref="U6"  Part="1"
-F 0 "U3" V 4500 3150 50  0000 C CNN
+F 0 "U6" V 4500 3150 50  0000 C CNN
 F 1 "74AC161" V 4300 3650 50  0000 C CNN
-F 2 "" H 4300 3650 50  0001 C CNN
+F 2 "Package_DIP:DIP-16_W7.62mm_Socket_LongPads" H 4300 3650 50  0001 C CNN
 F 3 "http://www.ti.com/lit/gpn/sn74LS161" H 4300 3650 50  0001 C CNN
 	1    4300 3650

Commit message: gpu sync board routed
Parts:
- U1, U2, U3: footprint Package_DIP:DIP-16_W7.62mm_Socket_LongPads -> Package_DIP:DIP-16_W7.62mm_Socket
Changed lines of the file:
@@
 EESchema Schematic File Version 4
-LIBS:Graphics-cache
-EELAYER 26 0
+EELAYER 29 0
 EELAYER END
 $Descr A4 11693 8268
 encoding utf-8
-Sheet 4 7
+Sheet 2 7
 Title ""
 Date ""
@@
 AR Path="/5CC1878B/5CC1EE88" Ref="#PWR0104"  Part="1"
 AR Path="/5CC8DF11/5CC1EE88" Ref="#PWR0121"  Part="1"
-F 0 "#PWR0121" H 8700 3500 50  0001 C CNN
+F 0 "#PWR0104" H 8700 3500 50  0001 C CNN
 F 1 "VCC" H 8717 3823 50  0000 C CNN
 F 2 "" H 8700 3650 50  0001 C CNN
@@
 AR Path="/5CC1878B/5CC1EE8E" Ref="U2"  Part="1"
 AR Path="/5CC8DF11/5CC1EE8E" Ref="U5"  Part="1"
-F 0 "U5" V 6300 3150 50  0000 C CNN
+F 0 "U2" V 6300 3150 50  0000 C CNN
 F 1 "74AC161" V 6100 3650 50  0000 C CNN
-F 2 "Package_DIP:DIP-16_W7.62mm_Socket_LongPads" H 6100 3650 50  0001 C CNN
+F 2 "Package_DIP:DIP-16_W7.62mm_Socket" H 6100 3650 50  0001 C CNN
 F 3 "http://www.ti.com/lit/gpn/sn74LS161" H 6100 3650 50  0001 C CNN
 	1    6100 3650
@@
 AR Path="/5CC1878B/5CC1EE94" Ref="U1"  Part="1"
 AR Path="/5CC8DF11/5CC1EE94" Ref="U4"  Part="1"
-F 0 "U4" V 8100 3150 50  0000 C CNN
+F 0 "U1" V 8100 3150 50  0000 C CNN
 F 1 "74AC161" V 7900 3650 50  0000 C CNN
-F 2 "Package_DIP:DIP-16_W7.62mm_Socket_LongPads" H 7900 3650 50  0001 C CNN
+F 2 "Package_DIP:DIP-16_W7.62mm_Socket" H 7900 3650 50  0001 C CNN
 F 3 "http://www.ti.com/lit/gpn/sn74LS161" H 7900 3650 50  0001 C CNN
 	1    7900 3650
@@
 AR Path="/5CC1878B/5CC1EEAF" Ref="#PWR0105"  Part="1"
 AR Path="/5CC8DF11/5CC1EEAF" Ref="#PWR0122"  Part="1"
-F 0 "#PWR0122" H 5300 3400 50  0001 C CNN
+F 0 "#PWR0105" H 5300 3400 50  0001 C CNN
 F 1 "GND" H 5305 3477 50  0000 C CNN
 F 2 "" H 5300 3650 50  0001 C CNN
@@
 AR Path="/5CC1878B/5CC1EEB5" Ref="#PWR0106"  Part="1"
 AR Path="/5CC8DF11/5CC1EEB5" Ref="#PWR0123"  Part="1"
-F 0 "#PWR0123" H 5100 3500 50  0001 C CNN
+F 0 "#PWR0106" H 5100 3500 50  0001 C CNN
 F 1 "VCC" H 5117 3823 50  0000 C CNN
 F 2 "" H 5100 3650 50  0001 C CNN
@@
 AR Path="/5CC1878B/5CC1EEBB" Ref="#PWR0107"  Part="1"
 AR Path="/5CC8DF11/5CC1EEBB" Ref="#PWR0124"  Part="1"
-F 0 "#PWR0124" H 7100 3400 50  0001 C CNN
+F 0 "#PWR0107" H 7100 3400 50  0001 C CNN
 F 1 "GND" H 7105 3477 50  0000 C CNN
 F 2 "" H 7100 3650 50  0001 C CNN
@@
 AR Path="/5CC1878B/5CC1EEC1" Ref="#PWR0108"  Part="1"
 AR Path="/5CC8DF11/5CC1EEC1" Ref="#PWR0125"  Part="1"
-F 0 "#PWR0125" H 3500 3400 50  0001 C CNN
+F 0 "#PWR0108" H 3500 3400 50  0001 C CNN
 F 1 "GND" H 3505 3477 50  0000 C CNN
 F 2 "" H 3500 3650 50  0001 C CNN
@@
 AR Path="/5CC1878B/5CC1EEC7" Ref="#PWR0109"  Part="1"
 AR Path="/5CC8DF11/5CC1EEC7" Ref="#PWR0126"  Part="1"
-F 0 "#PWR0126" H 6900 3500 50  0001 C CNN
+F 0 "#PWR0109" H 6900 3500 50  0001 C CNN
 F 1 "VCC" H 6917 3823 50  0000 C CNN
 F 2 "" H 6900 3650 50  0001 C CNN
@@
 AR Path="/5CC1878B/5CC1EED5" Ref="#PWR0110"  Part="1"
 AR Path="/5CC8DF11/5CC1EED5" Ref="#PWR0127"  Part="1"
-F 0 "#PWR0127" H 5900 2400 50  0001 C CNN
+F 0 "#PWR0110" H 5900 2400 50  0001 C CNN
 F 1 "VCC" H 5917 2723 50  0000 C CNN
 F 2 "" H 5900 2550 50  0001 C CNN
@@
 AR Path="/5CC1878B/5CC1EEE8" Ref="#PWR0111"  Part="1"
 AR Path="/5CC8DF11/5CC1EEE8" Ref="#PWR0128"  Part="1"
-F 0 "#PWR0128" H 4500 2300 50  0001 C CNN
+F 0 "#PWR0111" H 4500 2300 50  0001 C CNN
 F 1 "VCC" H 4517 2623 50  0000 C CNN
 F 2 "" H 4500 2450 50  0001 C CNN
@@
 AR Path="/5CC1878B/5CC1EEEE" Ref="U3"  Part="1"
 AR Path="/5CC8DF11/5CC1EEEE" Ref="U6"  Part="1"
-F 0 "U6" V 4500 3150 50  0000 C CNN
+F 0 "U3" V 4500 3150 50  0000 C CNN
 F 1 "74AC161" V 4300 3650 50  0000 C CNN
-F 2 "Package_DIP:DIP-16_W7.62mm_Socket_LongPads" H 4300 3650 50  0001 C CNN
+F 2 "Package_DIP:DIP-16_W7.62mm_Socket" H 4300 3650 50  0001 C CNN
 F 3 "http://www.ti.com/lit/gpn/sn74LS161" H 4300 3650 50  0001 C CNN
 	1    4300 3650
@@
 AR Path="/5CC1878B/5CC26AF1" Ref="#PWR0112"  Part="1"
 AR Path="/5CC8DF11/5CC26AF1" Ref="#PWR0129"  Part="1"
-F 0 "#PWR0129" H 7800 2400 50  0001 C CNN
+F 0 "#PWR0112" H 7800 2400 50  0001 C CNN
 F 1 "VCC" H 7817 2723 50  0000 C CNN
 F 2 "" H 7800 2550 50  0001 C CNN
