File: gpu-sync/Graphics.sch (KiCad schematic (older format))
At the start: 16 parts, among them J1 C96ABC, J2 Conn_01x26_Male, SW1 SW_Coded_SH-7050, U15 74HC04, U18 74LS573, U19 74LS573, U20 74LS573, U29 74HC688, U30 74AC138, U31 74AC138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

Commit message: gpu sync board component placement
Parts:
- removed X1: 25.175MHz, Oscillator:Oscillator_DIP-14, symbol Oscillator:CXO_DIP14
- added C1: CP_Small, Capacitor_THT:CP_Radial_D5.0mm_P2.00mm, symbol Device:CP_Small
- added C10, C11, C12, C13, C14, C15, C16, C17, C18, C19, C2, C20, C21, C22, C23, C24, C25, C3, C4, C5, C6, C7, C8, C9: C_Small, Capacitor_THT:C_Disc_D7.0mm_W2.5mm_P5.00mm, symbol Device:C_Small
- added X1: 25.175MHz, Oscillator:Oscillator_DIP-8_LargePads, symbol Oscillator:CXO_DIP8
- J1: footprint (none) -> common:Socket_DIN41612-CaseC1-full-Male-96Pin-3rows
- J2: footprint (none) -> Connector_IDC:IDC-Header_2x13_P2.54mm_Horizontal
- R1, R2, R3, R4: footprint (none) -> Resistor_THT:R_Axial_DIN0207_L6.3mm_D2.5mm_P10.16mm_Horizontal
- SW1: footprint (none) -> Button_Switch_THT:Nidec_Copal_SH-7010C
- U15, U34: footprint (none) -> Package_DIP:DIP-14_W7.62mm_Socket_LongPads
- U18, U19, U20: value 74LS573 -> 74AC573; footprint (none) -> Package_DIP:DIP-20_W7.62mm_Socket_LongPads
- U29: footprint (none) -> Package_DIP:DIP-20_W7.62mm_Socket_LongPads
- U30, U31: footprint (none) -> Package_DIP:DIP-16_W7.62mm_Socket_LongPads
Connections:
- no-connect marks 78 -> 81

Commit message: gpu sync board routed
Parts:
- added unit 7 of U15
- added U16, U17: 74HC109, Package_DIP:DIP-16_W7.62mm_Socket, symbol Graphics-rescue:74LS109-74xx
- added U32, U33: 74HC00, Package_DIP:DIP-14_W7.62mm_Socket, symbol 74xx:74HC00
- added unit 5 of U34
- U15, U34: footprint Package_DIP:DIP-14_W7.62mm_Socket_LongPads -> Package_DIP:DIP-14_W7.62mm_Socket
- U18, U19, U20, U29: footprint Package_DIP:DIP-20_W7.62mm_Socket_LongPads -> Package_DIP:DIP-20_W7.62mm_Socket
- U30, U31: footprint Package_DIP:DIP-16_W7.62mm_Socket_LongPads -> Package_DIP:DIP-16_W7.62mm_Socket
Connections:
- wire segments 334 -> 331
- no-connect marks 81 -> 82
