File: gpu-sync/cmpff.sch (KiCad schematic (older format))
At the start: 7 parts, among them U15 74HC04, U16 74HC109, U21 74AC573, U22 74AC573, U33 74HC00, U7 74HC688, U8 74HC688

Commit message: gpu sync board component placement
Parts:
- U15, U33: footprint (none) -> Package_DIP:DIP-14_W7.62mm_Socket_LongPads
- U16: footprint (none) -> Package_DIP:DIP-16_W7.62mm_Socket_LongPads
- U21, U22, U7, U8: footprint (none) -> Package_DIP:DIP-20_W7.62mm_Socket_LongPads
Changed lines of the file:
@@
 $Descr A4 11693 8268
 encoding utf-8
-Sheet 3 7
+Sheet 5 7
 Title ""
 Date ""
@@
 AR Path="/5CC9C16E/5CC72C3E" Ref="U11"  Part="1"
 AR Path="/5CCB1612/5CC72C3E" Ref="U13"  Part="1"
-F 0 "U7" H 6200 1750 50  0000 L CNN
+F 0 "U13" H 6200 1750 50  0000 L CNN
 F 1 "74HC688" V 6050 2750 50  0000 C CNN
-F 2 "" H 6050 2650 50  0001 C CNN
+F 2 "Package_DIP:DIP-20_W7.62mm_Socket_LongPads" H 6050 2650 50  0001 C CNN
 F 3 "http://www.ti.com/lit/gpn/sn74LS688" H 6050 2650 50  0001 C CNN
 	1    6050 2650
@@
 AR Path="/5CC9C16E/5CC72C44" Ref="U12"  Part="1"
 AR Path="/5CCB1612/5CC72C44" Ref="U14"  Part="1"
-F 0 "U8" H 6200 4600 50  0000 L CNN
+F 0 "U14" H 6200 4600 50  0000 L CNN
 F 1 "74HC688" V 6050 5600 50  0000 C CNN
-F 2 "" H 6050 5500 50  0001 C CNN
+F 2 "Package_DIP:DIP-20_W7.62mm_Socket_LongPads" H 6050 5500 50  0001 C CNN
 F 3 "http://www.ti.com/lit/gpn/sn74LS688" H 6050 5500 50  0001 C CNN
 	1    6050 5500
@@
 $Comp
 L Graphics-rescue:74LS109-74xx U?
-U 1 1 5CC72C4A
+U 2 1 5CC72C4A
 P 7050 2650
 AR Path="/5CC72C4A" Ref="U?"  Part="1"
@@
 AR Path="/5CC9C16E/5CC72C4A" Ref="U17"  Part="1"
 AR Path="/5CCB1612/5CC72C4A" Ref="U17"  Part="2"
-F 0 "U16" H 6900 2350 50  0000 R CNN
+F 0 "U17" H 6900 2350 50  0000 R CNN
 F 1 "74HC109" V 7150 2400 50  0000 R CNN
-F 2 "" H 7050 2650 50  0001 C CNN
+F 2 "Package_DIP:DIP-16_W7.62mm_Socket_LongPads" H 7050 2650 50  0001 C CNN
 F 3 "http://www.ti.com/lit/gpn/sn74LS109" H 7050 2650 50  0001 C CNN
-	1    7050 2650
+	2    7050 2650
 	1    0    0    -1
 $EndComp
 $Comp
 L 74xx:74HC04 U?
-U 2 1 5CC72C50
+U 5 1 5CC72C50
 P 6650 2150
 AR Path="/5CC72C50" Ref="U?"  Part="1"
@@
 F 0 "U15" V 6450 2300 50  0000 C CNN
 F 1 "74HC04" V 6750 2350 50  0000 C CNN
-F 2 "" H 6650 2150 50  0001 C CNN
+F 2 "Package_DIP:DIP-14_W7.62mm_Socket_LongPads" H 6650 2150 50  0001 C CNN
 F 3 "https://assets.nexperia.com/documents/data-sheet/74HC_HCT04.pdf" H 6650 2150 50  0001 C CNN
-	2    6650 2150
+	5    6650 2150
 	0    1    1    0
 $EndComp
@@
 AR Path="/5CC9C16E/5CE3CB3C" Ref="U25"  Part="1"
 AR Path="/5CCB1612/5CE3CB3C" Ref="U27"  Part="1"
-F 0 "U21" H 3650 3450 50  0000 C CNN
+F 0 "U27" H 3650 3450 50  0000 C CNN
 F 1 "74AC573" H 3650 2850 50  0000 C CNN
-F 2 "" H 3650 3150 50  0001 C CNN
+F 2 "Package_DIP:DIP-20_W7.62mm_Socket_LongPads" H 3650 3150 50  0001 C CNN
 F 3 "74xx/74hc573.pdf" H 3650 3150 50  0001 C CNN
 	1    3650 3150
@@
 AR Path="/5CC9C16E/5CE46B72" Ref="U26"  Part="1"
 AR Path="/5CCB1612/5CE46B72" Ref="U28"  Part="1"
-F 0 "U22" H 3650 6300 50  0000 C CNN
+F 0 "U28" H 3650 6300 50  0000 C CNN
 F 1 "74AC573" H 3650 5700 50  0000 C CNN
-F 2 "" H 3650 6000 50  0001 C CNN
+F 2 "Package_DIP:DIP-20_W7.62mm_Socket_LongPads" H 3650 6000 50  0001 C CNN
 F 3 "74xx/74hc573.pdf" H 3650 6000 50  0001 C CNN
 	1    3650 6000
@@
 $Comp
 L 74xx:74HC00 U?
-U 1 1 5D446A15
+U 3 1 5D446A15
 P 2750 3550
 AR Path="/5D446A15" Ref="U?"  Part="1"
@@
 AR Path="/5CC6FF8F/5D446A15" Ref="U32"  Part="1"
 AR Path="/5CC85C26/5D446A15" Ref="U32"  Part="3"
-F 0 "U32" H 2600 3750 50  0000 L CNN
+F 0 "U33" H 2600 3750 50  0000 L CNN
 F 1 "74HC00" H 2550 3300 50  0000 L CNN
-F 2 "" H 2750 3550 50  0001 C CNN
+F 2 "Package_DIP:DIP-14_W7.62mm_Socket_LongPads" H 2750 3550 50  0001 C CNN
 F 3 "http://www.ti.com/lit/gpn/sn74hc00" H 2750 3550 50  0001 C CNN
-	1    2750 3550
+	3    2750 3550
 	1    0    0    -1
 $EndComp
@@
 $Comp
 L 74xx:74HC00 U?
-U 2 1 5D44D4F0
+U 4 1 5D44D4F0
 P 2750 6400
 AR Path="/5D44D4F0" Ref="U?"  Part="1"
@@
 AR Path="/5CC6FF8F/5D44D4F0" Ref="U32"  Part="2"
 AR Path="/5CC85C26/5D44D4F0" Ref="U32"  Part="4"
-F 0 "U32" H 2600 6600 50  0000 L CNN
+F 0 "U33" H 2600 6600 50  0000 L CNN
 F 1 "74HC00" H 2550 6150 50  0000 L CNN
-F 2 "" H 2750 6400 50  0001 C CNN
+F 2 "Package_DIP:DIP-14_W7.62mm_Socket_LongPads" H 2750 6400 50  0001 C CNN
 F 3 "http://www.ti.com/lit/gpn/sn74hc00" H 2750 6400 50  0001 C CNN
-	2    2750 6400
-	1    0    0    -1
-$EndComp
+	4    2750 6400
+	1    0    0    -1
+$EndComp

Commit message: gpu sync board routed
Parts:
- U15, U33: footprint Package_DIP:DIP-14_W7.62mm_Socket_LongPads -> Package_DIP:DIP-14_W7.62mm_Socket
- U16: footprint Package_DIP:DIP-16_W7.62mm_Socket_LongPads -> Package_DIP:DIP-16_W7.62mm_Socket
- U21, U22, U7, U8: footprint Package_DIP:DIP-20_W7.62mm_Socket_LongPads -> Package_DIP:DIP-20_W7.62mm_Socket
Changed lines of the file:
@@
 EESchema Schematic File Version 4
-LIBS:Graphics-cache
-EELAYER 26 0
+EELAYER 29 0
 EELAYER END
 $Descr A4 11693 8268
@@
 AR Path="/5CC9C16E/5CC72C3E" Ref="U11"  Part="1"
 AR Path="/5CCB1612/5CC72C3E" Ref="U13"  Part="1"
-F 0 "U13" H 6200 1750 50  0000 L CNN
+F 0 "U11" H 6200 1750 50  0000 L CNN
 F 1 "74HC688" V 6050 2750 50  0000 C CNN
-F 2 "Package_DIP:DIP-20_W7.62mm_Socket_LongPads" H 6050 2650 50  0001 C CNN
+F 2 "Package_DIP:DIP-20_W7.62mm_Socket" H 6050 2650 50  0001 C CNN
 F 3 "http://www.ti.com/lit/gpn/sn74LS688" H 6050 2650 50  0001 C CNN
 	1    6050 2650
@@
 AR Path="/5CC9C16E/5CC72C44" Ref="U12"  Part="1"
 AR Path="/5CCB1612/5CC72C44" Ref="U14"  Part="1"
-F 0 "U14" H 6200 4600 50  0000 L CNN
+F 0 "U12" H 6200 4600 50  0000 L CNN
 F 1 "74HC688" V 6050 5600 50  0000 C CNN
-F 2 "Package_DIP:DIP-20_W7.62mm_Socket_LongPads" H 6050 5500 50  0001 C CNN
+F 2 "Package_DIP:DIP-20_W7.62mm_Socket" H 6050 5500 50  0001 C CNN
 F 3 "http://www.ti.com/lit/gpn/sn74LS688" H 6050 5500 50  0001 C CNN
 	1    6050 5500
@@
 $Comp
 L Graphics-rescue:74LS109-74xx U?
-U 2 1 5CC72C4A
+U 1 1 5CC72C4A
 P 7050 2650
 AR Path="/5CC72C4A" Ref="U?"  Part="1"
@@
 F 0 "U17" H 6900 2350 50  0000 R CNN
 F 1 "74HC109" V 7150 2400 50  0000 R CNN
-F 2 "Package_DIP:DIP-16_W7.62mm_Socket_LongPads" H 7050 2650 50  0001 C CNN
+F 2 "Package_DIP:DIP-16_W7.62mm_Socket" H 7050 2650 50  0001 C CNN
 F 3 "http://www.ti.com/lit/gpn/sn74LS109" H 7050 2650 50  0001 C CNN
-	2    7050 2650
+	1    7050 2650
 	1    0    0    -1
 $EndComp
 $Comp
 L 74xx:74HC04 U?
-U 5 1 5CC72C50
+U 4 1 5CC72C50
 P 6650 2150
 AR Path="/5CC72C50" Ref="U?"  Part="1"
@@
 F 0 "U15" V 6450 2300 50  0000 C CNN
 F 1 "74HC04" V 6750 2350 50  0000 C CNN
-F 2 "Package_DIP:DIP-14_W7.62mm_Socket_LongPads" H 6650 2150 50  0001 C CNN
+F 2 "Package_DIP:DIP-14_W7.62mm_Socket" H 6650 2150 50  0001 C CNN
 F 3 "https://assets.nexperia.com/documents/data-sheet/74HC_HCT04.pdf" H 6650 2150 50  0001 C CNN
-	5    6650 2150
+	4    6650 2150
 	0    1    1    0
 $EndComp
@@
 AR Path="/5CC9C16E/5CC72C5A" Ref="#PWR0130"  Part="1"
 AR Path="/5CCB1612/5CC72C5A" Ref="#PWR0134"  Part="1"
-F 0 "#PWR0117" H 6050 3600 50  0001 C CNN
+F 0 "#PWR0130" H 6050 3600 50  0001 C CNN
 F 1 "GND" H 6055 3677 50  0000 C CNN
 F 2 "" H 6050 3850 50  0001 C CNN
@@
 AR Path="/5CC9C16E/5CC72C60" Ref="#PWR0131"  Part="1"
 AR Path="/5CCB1612/5CC72C60" Ref="#PWR0135"  Part="1"
-F 0 "#PWR0118" H 6050 6450 50  0001 C CNN
+F 0 "#PWR0131" H 6050 6450 50  0001 C CNN
 F 1 "GND" H 6055 6527 50  0000 C CNN
 F 2 "" H 6050 6700 50  0001 C CNN
@@
 AR Path="/5CC9C16E/5CC72C66" Ref="#PWR0132"  Part="1"
 AR Path="/5CCB1612/5CC72C66" Ref="#PWR0136"  Part="1"
-F 0 "#PWR0119" H 6050 4150 50  0001 C CNN
+F 0 "#PWR0132" H 6050 4150 50  0001 C CNN
 F 1 "VCC" H 6067 4473 50  0000 C CNN
 F 2 "" H 6050 4300 50  0001 C CNN
@@
 AR Path="/5CC9C16E/5CC72C6C" Ref="#PWR0133"  Part="1"
 AR Path="/5CCB1612/5CC72C6C" Ref="#PWR0137"  Part="1"
-F 0 "#PWR0120" H 6050 1300 50  0001 C CNN
+F 0 "#PWR0133" H 6050 1300 50  0001 C CNN
 F 1 "VCC" H 6067 1623 50  0000 C CNN
 F 2 "" H 6050 1450 50  0001 C CNN
@@
 AR Path="/5CC9C16E/5CE3CB3C" Ref="U25"  Part="1"
 AR Path="/5CCB1612/5CE3CB3C" Ref="U27"  Part="1"
-F 0 "U27" H 3650 3450 50  0000 C CNN
+F 0 "U25" H 3650 3450 50  0000 C CNN
 F 1 "74AC573" H 3650 2850 50  0000 C CNN
-F 2 "Package_DIP:DIP-20_W7.62mm_Socket_LongPads" H 3650 3150 50  0001 C CNN
+F 2 "Package_DIP:DIP-20_W7.62mm_Socket" H 3650 3150 50  0001 C CNN
 F 3 "74xx/74hc573.pdf" H 3650 3150 50  0001 C CNN
 	1    3650 3150
@@
 AR Path="/5CC9C16E/5CE46B72" Ref="U26"  Part="1"
 AR Path="/5CCB1612/5CE46B72" Ref="U28"  Part="1"
-F 0 "U28" H 3650 6300 50  0000 C CNN
+F 0 "U26" H 3650 6300 50  0000 C CNN
 F 1 "74AC573" H 3650 5700 50  0000 C CNN
-F 2 "Package_DIP:DIP-20_W7.62mm_Socket_LongPads" H 3650 6000 50  0001 C CNN
+F 2 "Package_DIP:DIP-20_W7.62mm_Socket" H 3650 6000 50  0001 C CNN
 F 3 "74xx/74hc573.pdf" H 3650 6000 50  0001 C CNN
 	1    3650 6000
@@
 AR Path="/5CC9C16E/5CE58AD7" Ref="#PWR0148"  Part="1"
 AR Path="/5CCB1612/5CE58AD7" Ref="#PWR0149"  Part="1"
-F 0 "#PWR0147" H 7050 2100 50  0001 C CNN
+F 0 "#PWR0148" H 7050 2100 50  0001 C CNN
 F 1 "VCC" H 7067 2423 50  0000 C CNN
 F 2 "" H 7050 2250 50  0001 C CNN
@@
 AR Path="/5CCB1612/5D30F4A4" Ref="#PWR0159"  Part="1"
 AR Path="/5CC85C26/5D30F4A4" Ref="#PWR0161"  Part="1"
-F 0 "#PWR0161" H 3100 3450 50  0001 C CNN
+F 0 "#PWR0157" H 3100 3450 50  0001 C CNN
 F 1 "GND" H 3105 3527 50  0000 C CNN
 F 2 "" H 3100 3700 50  0001 C CNN
@@
 AR Path="/5CCB1612/5D313614" Ref="#PWR0160"  Part="1"
 AR Path="/5CC85C26/5D313614" Ref="#PWR0162"  Part="1"
-F 0 "#PWR0162" H 3100 6300 50  0001 C CNN
+F 0 "#PWR0158" H 3100 6300 50  0001 C CNN
 F 1 "GND" H 3105 6377 50  0000 C CNN
 F 2 "" H 3100 6550 50  0001 C CNN
@@
 $Comp
 L 74xx:74HC00 U?
-U 3 1 5D446A15
+U 1 1 5D446A15
 P 2750 3550
 AR Path="/5D446A15" Ref="U?"  Part="1"
@@
 F 0 "U33" H 2600 3750 50  0000 L CNN
 F 1 "74HC00" H 2550 3300 50  0000 L CNN
-F 2 "Package_DIP:DIP-14_W7.62mm_Socket_LongPads" H 2750 3550 50  0001 C CNN
+F 2 "Package_DIP:DIP-14_W7.62mm_Socket" H 2750 3550 50  0001 C CNN
 F 3 "http://www.ti.com/lit/gpn/sn74hc00" H 2750 3550 50  0001 C CNN
-	3    2750 3550
+	1    2750 3550
 	1    0    0    -1
 $EndComp
@@
 $Comp
 L 74xx:74HC00 U?
-U 4 1 5D44D4F0
+U 2 1 5D44D4F0
 P 2750 6400
 AR Path="/5D44D4F0" Ref="U?"  Part="1"
@@
 F 0 "U33" H 2600 6600 50  0000 L CNN
 F 1 "74HC00" H 2550 6150 50  0000 L CNN
-F 2 "Package_DIP:DIP-14_W7.62mm_Socket_LongPads" H 2750 6400 50  0001 C CNN
+F 2 "Package_DIP:DIP-14_W7.62mm_Socket" H 2750 6400 50  0001 C CNN
 F 3 "http://www.ti.com/lit/gpn/sn74hc00" H 2750 6400 50  0001 C CNN
-	4    2750 6400
+	2    2750 6400
 	1    0    0    -1
 $EndComp
@@
 AR Path="/5CCB1612/5EC996EF" Ref="#PWR0180"  Part="1"
 AR Path="/5CC85C26/5EC996EF" Ref="#PWR0182"  Part="1"
-F 0 "#PWR0182" H 3650 5050 50  0001 C CNN
+F 0 "#PWR0178" H 3650 5050 50  0001 C CNN
 F 1 "VCC" H 3667 5373 50  0000 C CNN
 F 2 "" H 3650 5200 50  0001 C CNN
@@
 AR Path="/5CCB1612/5EC99768" Ref="#PWR0181"  Part="1"
 AR Path="/5CC85C26/5EC99768" Ref="#PWR0183"  Part="1"
-F 0 "#PWR0183" H 3650 6550 50  0001 C CNN
+F 0 "#PWR0179" H 3650 6550 50  0001 C CNN
 F 1 "GND" H 3655 6627 50  0000 C CNN
 F 2 "" H 3650 6800 50  0001 C CNN
@@
 AR Path="/5CCB1612/5EC99821" Ref="#PWR0188"  Part="1"
 AR Path="/5CC85C26/5EC99821" Ref="#PWR0190"  Part="1"
-F 0 "#PWR0190" H 3650 2200 50  0001 C CNN
+F 0 "#PWR0186" H 3650 2200 50  0001 C CNN
 F 1 "VCC" H 3667 2523 50  0000 C CNN
 F 2 "" H 3650 2350 50  0001 C CNN
@@
 AR Path="/5CCB1612/5EC99885" Ref="#PWR0189"  Part="1"
 AR Path="/5CC85C26/5EC99885" Ref="#PWR0191"  Part="1"
-F 0 "#PWR0191" H 3650 3700 50  0001 C CNN
+F 0 "#PWR0187" H 3650 3700 50  0001 C CNN
 F 1 "GND" H 3655 3777 50  0000 C CNN
 F 2 "" H 3650 3950 50  0001 C CNN
