File: memory/memory.kicad_pcb (KiCad board)
At the start: 2 copper layers, 160 x 100 mm, 19 parts, among them J1 C96ABC, J2 Conn_02x08_Odd_Even, U1 LY62256PL-55LLI, U2 LY62256PL-55LLI, U3 74AC138, U4 74HC00, U5 74HC595

Commit message: layout memory
Parts:
- moved BT1 230.0 mm to (105.6, 60.6), turned to 270 degrees
- moved U3 214.9 mm to (133.6, 121.6)
- moved C6 212.8 mm to (157.7, 60.6), turned to 90 degrees
- moved U4 210.6 mm to (148.8, 121.6)
- moved JP1 208.3 mm to (156.4, 77.1)
- moved U5 206.3 mm to (174.2, 121.6)
- moved C3 187.2 mm to (139.8, 116.5), turned to 180 degrees
- moved J2 180.0 mm to (164.1, 121.6)
- moved U1 167.6 mm to (133.6, 74.6)
- moved C1 164.1 mm to (143.7, 69.5), turned to 180 degrees
- moved C4 164.1 mm to (155.1, 116.5), turned to 180 degrees
- moved R1 157.3 mm to (152.6, 65.7)
- moved D1 153.7 mm to (145.0, 60.6), turned to 180 degrees
- moved U2 153.3 mm to (166.6, 74.6)
- moved C2 146.4 mm to (176.8, 69.5), turned to 180 degrees
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Connections:
- J2 pad 1: Net-(J2-Pad1) -> ~WAIT
- J2 pad 10: ~WAIT -> Net-(J2-Pad10)
- J2 pad 11: Net-(J2-Pad11) -> ~WAIT
- J2 pad 12: ~WAIT -> Net-(J2-Pad12)
- J2 pad 13: Net-(J2-Pad13) -> ~WAIT
- J2 pad 14: ~WAIT -> Net-(J2-Pad14)
- J2 pad 15: Net-(J2-Pad15) -> ~WAIT
- J2 pad 16: ~WAIT -> Net-(J2-Pad16)
- J2 pad 2: ~WAIT -> Net-(J2-Pad2)
- J2 pad 3: Net-(J2-Pad3) -> ~WAIT
- J2 pad 4: ~WAIT -> Net-(J2-Pad4)
- J2 pad 5: Net-(J2-Pad5) -> ~WAIT
- J2 pad 6: ~WAIT -> Net-(J2-Pad6)
- J2 pad 7: Net-(J2-Pad7) -> ~WAIT
- J2 pad 8: ~WAIT -> Net-(J2-Pad8)
- J2 pad 9: Net-(J2-Pad9) -> ~WAIT
- JP1 pad 1: D0 -> Net-(JP1-Pad1)
- R2 pad 2: D0 -> Net-(JP1-Pad1)
- U1 pad 27: D0 -> Net-(JP1-Pad1)
- U5 pad 1: Net-(J2-Pad3) -> Net-(J2-Pad4)
- U5 pad 15: Net-(J2-Pad1) -> Net-(J2-Pad2)
- U5 pad 2: Net-(J2-Pad5) -> Net-(J2-Pad6)
- U5 pad 3: Net-(J2-Pad7) -> Net-(J2-Pad8)
- U5 pad 4: Net-(J2-Pad9) -> Net-(J2-Pad10)
- U5 pad 5: Net-(J2-Pad11) -> Net-(J2-Pad12)
- U5 pad 6: Net-(J2-Pad13) -> Net-(J2-Pad14)
- U5 pad 7: Net-(J2-Pad15) -> Net-(J2-Pad16)
Routing:
- net GND: track 0.00 -> 448.4 mm
- net VMEM: track 0.00 -> 192.5 mm
- net ~ROB: track 0.00 -> 171.2 mm
- net +BATT: track 0.00 -> 151.1 mm
- net A12: track 0.00 -> 111.4 mm, vias 0 -> 1
- net A13: track 0.00 -> 106.0 mm, vias 0 -> 2
- net A9: track 0.00 -> 103.9 mm, vias 0 -> 3
- net A14: track 0.00 -> 103.9 mm
- net D2: track 0.00 -> 99.1 mm, vias 0 -> 1
- net D0: track 0.00 -> 97.6 mm, vias 0 -> 1
- net ~WAIT: track 0.00 -> 94.7 mm, vias 0 -> 2
- net D3: track 0.00 -> 91.8 mm, vias 0 -> 1
- net D5: track 0.00 -> 90.4 mm, vias 0 -> 1
- net A0: track 0.00 -> 89.7 mm, vias 0 -> 1
- net D4: track 0.00 -> 87.5 mm, vias 0 -> 1
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- added copper zone on B.Cu, net GND
- added copper zone on F.Cu, net GND
