File: cpu-new/cpu-new.kicad_pcb (KiCad board)
At the start: 2 copper layers, 160 x 100 mm, 61 parts, among them J1 Barrel_Jack, J2 C96ABC, SW1 SW_Push, SW2 SW_SPDT, U1 Z84C0010PEG, U10 74AC10, U11 74AC14, U12 L7805, U2 LY62256PL-55LLI, U3 LY62256PL-55LLI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

Commit message: routing
Routing:
- net Net-(SW2-Pad3): track 46.5 -> 175.5 mm, vias 1 -> 2
- net Net-(U1-Pad31): track 19.0 -> 126.5 mm
- net Net-(U1-Pad33): track 29.8 -> 126.6 mm
- net Net-(U1-Pad35): track 35.3 -> 122.1 mm, vias 1 -> 2
- net Net-(U1-Pad36): track 37.8 -> 123.9 mm, vias 1 -> 2
- net Net-(U1-Pad21): track 78.1 -> 157.6 mm, vias 1 -> 2
- net Net-(U1-Pad32): track 24.6 -> 91.2 mm
- net Net-(U1-Pad30): track 13.0 -> 79.7 mm
- net Net-(U1-Pad34): track 32.7 -> 99.4 mm
- net Net-(U1-Pad37): track 41.4 -> 107.0 mm
- net Net-(U1-Pad7): track 42.6 -> 105.3 mm, vias 0 -> 2
- net Net-(U1-Pad4): track 107.4 -> 163.0 mm, vias 1 -> 2
- net Net-(U1-Pad8): track 38.5 -> 93.7 mm, vias 0 -> 1
- net Net-(U1-Pad14): track 47.4 -> 100.9 mm, vias 1 -> 2
- net Net-(U1-Pad15): track 51.2 -> 103.7 mm, vias 1 -> 2
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